File: bitaxeGamma.kicad_sch (KiCad schematic)
At the start: 20 parts, among them J1 54-00164

Commit message: mounting holes to 3mm
Parts:
- H5, H6, H7, H8: footprint MountingHole:MountingHole_3.2mm_M3_Pad -> MountingHole:MountingHole_3mm_Pad
Changed lines of the file:
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@@
 			)
 		)
-		(property "Footprint" "MountingHole:MountingHole_3.2mm_M3_Pad"
+		(property "Footprint" "MountingHole:MountingHole_3mm_Pad"
 			(at 66.04 186.69 0)
 			(effects
@@
 			)
 		)
-		(property "Footprint" "MountingHole:MountingHole_3.2mm_M3_Pad"
+		(property "Footprint" "MountingHole:MountingHole_3mm_Pad"
 			(at 66.04 180.34 0)
 			(effects
@@
 			)
 		)
-		(property "Footprint" "MountingHole:MountingHole_3.2mm_M3_Pad"
+		(property "Footprint" "MountingHole:MountingHole_3mm_Pad"
 			(at 66.04 173.99 0)
 			(effects
@@
 			)
 		)
-		(property "Footprint" "MountingHole:MountingHole_3.2mm_M3_Pad"
+		(property "Footprint" "MountingHole:MountingHole_3mm_Pad"
 			(at 66.04 167.64 0)
 			(effects

Commit message: update worksheet
Other:
- company: (none) -> bitaxeorg
Changed lines of the file:
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@@
 		(date "2025-04-29")
 		(rev "603")
+		(company "bitaxeorg")
+		(comment 1 "OHLv2")
 	)
 	(junction
@@
 					(size 1.27 1.27)
 				)
-			)
-		)
+				(hide yes)
+			)
+		)
