File: bitaxeGamma.kicad_sch (KiCad schematic)
At the start: 20 parts, among them J1 54-00164

Commit message: eco-603-impl: schematic ECO (E0-E6, R2-R3)
E0 #6/8bd74c8: R21 removed, U9.8 to 1V2, U9.9 direct GND.
E1 #47: U2 SYNC/BCX_CLK/BCX_DAT to AGND.
E2 #25 + R2: R30-R32 4k7 PMBus, R35 10k PGD pull-ups.
E3 #13/#16: R22/R23 100R to 10R.
E4 #11/#17: F1 5A series, D1 SMAJ5.0A, C60 bulk.
E5 #37 + R3: R33/R34 5k1 CC, D2/D5 USB ESD, D3/D4 I2C ESD.
R3: C61 47u + C62 100n PVIN/AVIN bulk.
Rev 601->603. ERC: 18->19 err (PVIN PWR flag side effect of F1,
same benign class); netlist-verified, geometry-audited.
Parts:
- added C60: 100uF, Capacitor_SMD:C_1206_3216Metric, symbol Device:C
- added D1: SMAJ5.0A, Diode_SMD:D_SMA, symbol bitaxe:TVS_BIDIR
- added F1: 5A, Fuse_SMD:Fuse_1206_3216Metric, symbol bitaxe:FUSE_2PIN
Connections:
- net 5V: now also C60.1, D1.1
- net GND: now also C60.2, D1.2
- net Power/VIN: now also F1.2; no longer J1.1
- new net: F1.1, J1.1
