File: fan.kicad_sch (KiCad schematic)
At the start: 14 parts, among them J6 Conn_01x04, U10 EMC2101

Commit message: update worksheet
Other:
- company: (none) -> bitaxeorg
Changed lines of the file:
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@@
 		(date "2025-04-29")
 		(rev "603")
+		(company "bitaxeorg")
+		(comment 1 "OHLv2")
 	)
 	(text "EMC2101 Controls the fan, and reads the ASIC chip temperature"
