File: fan.kicad_sch (KiCad schematic)
At the start: 15 parts, among them J6 Conn_01x04, J7 Conn_01x04, U10 EMC2101

Commit message: eco-603-impl: schematic ECO (E0-E6, R2-R3)
E0 #6/8bd74c8: R21 removed, U9.8 to 1V2, U9.9 direct GND.
E1 #47: U2 SYNC/BCX_CLK/BCX_DAT to AGND.
E2 #25 + R2: R30-R32 4k7 PMBus, R35 10k PGD pull-ups.
E3 #13/#16: R22/R23 100R to 10R.
E4 #11/#17: F1 5A series, D1 SMAJ5.0A, C60 bulk.
E5 #37 + R3: R33/R34 5k1 CC, D2/D5 USB ESD, D3/D4 I2C ESD.
R3: C61 47u + C62 100n PVIN/AVIN bulk.
Rev 601->603. ERC: 18->19 err (PVIN PWR flag side effect of F1,
same benign class); netlist-verified, geometry-audited.
Parts:
- R22, R23: value 100 -> 10; DK 311-100LRCT-ND -> 311-10.0LRCT-ND; PARTNO RC0402FR-07100RL -> RC0402FR-0710RL
Changed lines of the file:
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@@
 	(title_block
 		(title "bitaxeGamma")
-		(date "2024-09-26")
-		(rev "601")
+		(date "2026-09-05")
+		(rev "603")
 	)
 	(text "EMC2101 Controls the fan, and reads the ASIC chip temperature"
@@
 			)
 		)
-		(property "Value" "100"
+		(property "Value" "10"
 			(at 94.615 79.88 0)
 			(effects
@@
 			)
 		)
-		(property "DK" "311-100LRCT-ND"
+		(property "DK" "311-10.0LRCT-ND"
 			(at 90.17 76.2 0)
 			(effects
@@
 			)
 		)
-		(property "PARTNO" "RC0402FR-07100RL"
+		(property "PARTNO" "RC0402FR-0710RL"
 			(at 90.17 76.2 0)
 			(effects
@@
 			)
 		)
-		(property "Value" "100"
+		(property "Value" "10"
 			(at 91.44 70.485 0)
 			(effects
@@
 			)
 		)
-		(property "DK" "311-100LRCT-ND"
+		(property "DK" "311-10.0LRCT-ND"
 			(at 91.44 73.66 0)
 			(effects
@@
 			)
 		)
-		(property "PARTNO" "RC0402FR-07100RL"
+		(property "PARTNO" "RC0402FR-0710RL"
 			(at 91.44 73.66 0)
 			(effects
