File: bm1370.kicad_sch (KiCad schematic)
At the start: 49 parts, among them U5 MCP1824T-1202E/OT, U6 MCP1824T-0802E, U7 25MHz, U8 BM1370_mode1, U9 SN74AVC4T774

Commit message: eco-603-impl: schematic ECO (E0-E6, R2-R3)
E0 #6/8bd74c8: R21 removed, U9.8 to 1V2, U9.9 direct GND.
E1 #47: U2 SYNC/BCX_CLK/BCX_DAT to AGND.
E2 #25 + R2: R30-R32 4k7 PMBus, R35 10k PGD pull-ups.
E3 #13/#16: R22/R23 100R to 10R.
E4 #11/#17: F1 5A series, D1 SMAJ5.0A, C60 bulk.
E5 #37 + R3: R33/R34 5k1 CC, D2/D5 USB ESD, D3/D4 I2C ESD.
R3: C61 47u + C62 100n PVIN/AVIN bulk.
Rev 601->603. ERC: 18->19 err (PVIN PWR flag side effect of F1,
same benign class); netlist-verified, geometry-audited.
Parts:
- removed R21: 20k, Resistor_SMD:R_0402_1005Metric, symbol Device:R_US
Connections:
- net 1V2: now also U9.8 (DIR4)
- net GND: now also U9.9 (OE); no longer U9.8 (DIR4)
Changed lines of the file:
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@@
 	(title_block
 		(title "bitaxeGamma")
-		(date "2024-09-26")
-		(rev "601")
+		(date "2026-09-05")
+		(rev "603")
 	)
 	(text "Reference Voltage Regulators"
@@
 	)
 	(junction
-		(at 193.04 59.69)
-		(diameter 0)
-		(color 0 0 0 0)
-	)
-	(junction
 		(at 140.97 85.09)
 		(diameter 0)
@@
 	(wire
 		(pts
-			(xy 193.04 59.69) (xy 193.04 57.15)
-		)
-		(stroke
-			(width 0)
-			(type default)
-		)
-	)
-	(wire
-		(pts
 			(xy 242.57 43.18) (xy 242.57 59.69)
 		)
@@
 	(wire
 		(pts
-			(xy 193.04 46.99) (xy 193.04 49.53)
-		)
-		(stroke
-			(width 0)
-			(type default)
-		)
-	)
-	(wire
-		(pts
 			(xy 224.79 46.99) (xy 229.87 46.99)
 		)
@@
 	(wire
 		(pts
-			(xy 204.47 46.99) (xy 193.04 46.99)
-		)
-		(stroke
-			(width 0)
-			(type default)
-		)
-	)
-	(wire
-		(pts
 			(xy 105.41 53.34) (xy 105.41 50.8)
 		)
@@
 	(wire
 		(pts
-			(xy 173.99 59.69) (xy 193.04 59.69)
-		)
-		(stroke
-			(width 0)
-			(type default)
-		)
-	)
-	(wire
-		(pts
 			(xy 49.53 172.72) (xy 50.8 172.72)
 		)
@@
 	(wire
 		(pts
-			(xy 198.12 59.69) (xy 193.04 59.69)
-		)
-		(stroke
-			(width 0)
-			(type default)
-		)
-	)
-	(wire
-		(pts
 			(xy 66.04 55.88) (xy 66.04 58.42)
 		)
@@
 		)
 	)
-	(label "GND"
+	(label "1V2"
 		(at 229.87 52.07 180)
 		(effects
@@
 	(symbol
 		(lib_id "Device:R_US")
-		(at 193.04 53.34 180)
-		(unit 1)
-		(exclude_from_sim no)
-		(in_bom yes)
-		(on_board yes)
-		(dnp no)
-		(property "Reference" "R21"
-			(at 188.595 52.07 0)
-			(effects
-				(font
-					(size 1.27 1.27)
-				)
-			)
-		)
-		(property "Value" "20k"
-			(at 188.595 54.61 0)
-			(effects
-				(font
-					(size 1.27 1.27)
-				)
-			)
-		)
-		(property "Footprint" "Resistor_SMD:R_0402_1005Metric"
-			(at 192.024 53.086 90)
-			(effects
-				(font
-					(size 1.27 1.27)
-				)
-				(hide yes)
-			)
-		)
-		(property "Datasheet" "~"
-			(at 193.04 53.34 0)
-			(effects
-				(font
-					(size 1.27 1.27)
-				)
-				(hide yes)
-			)
-		)
-		(property "Description" ""
-			(at 193.04 53.34 0)
-			(effects
-				(font
-					(size 1.27 1.27)
-				)
-				(hide yes)
-			)
-		)
-		(property "DK" "311-20.0KLRCT-ND"
-			(at 193.04 53.34 0)
-			(effects
-				(font
-					(size 1.27 1.27)
-				)
-				(hide yes)
-			)
-		)
-		(property "PARTNO" "RC0402FR-0720KL"
-			(at 193.04 53.34 0)
-			(effects
-				(font
-					(size 1.27 1.27)
-				)
-				(hide yes)
-			)
-		)
-		(pin "1"
-		)
-		(pin "2"
-		)
-		(instances
-			(project "bitaxeGamma"
-				(path "/e63e39d7-6ac0-4ffd-8aa3-1841a4541b55/4cf9c075-d009-4c35-9949-adda70ae20c7"
-					(reference "R21")
-					(unit 1)
-				)
-			)
-		)
-	)
-	(symbol
-		(lib_id "Device:R_US")
 		(at 81.28 137.16 180)
 		(unit 1)
@@
 		)
 	)
+	(wire
+		(pts
+			(xy 204.47 46.99) (xy 198.12 46.99)
+		)
+		(stroke
+			(width 0)
+			(type default)
+		)
+	)
+	(wire
+		(pts
+			(xy 198.12 46.99) (xy 198.12 52.07)
+		)
+		(stroke
+			(width 0)
+			(type default)
+		)
+	)
+	(wire
+		(pts
+			(xy 173.99 59.69) (xy 198.12 59.69)
+		)
+		(stroke
+			(width 0)
+			(type default)
+		)
+	)
+	(junction
+		(at 198.12 52.07)
+		(diameter 0)
+		(color 0 0 0 0)
+	)
 )
